Commit message: Added gazebo velocity controllers

File: crazyflie_description/urdf/crazyflie_basic.urdf (robot description, URDF)
Before this commit: robot crazyflie, 6 links, 5 joints
Links:
- removed link dummy
Joints:
- removed joint dummy_joint
- joint crazyflie_M1_joint: limit lower=-1e+16 upper=1e+16 effort=-1 velocity=-1 -> lower=-1e+16 upper=1e+16 effort=1000 velocity=100
- joint crazyflie_M2_joint: limit lower=-1e+16 upper=1e+16 effort=-1 velocity=-1 -> lower=-1e+16 upper=1e+16 effort=1000 velocity=100
- joint crazyflie_M3_joint: limit lower=-1e+16 upper=1e+16 effort=-1 velocity=-1 -> lower=-1e+16 upper=1e+16 effort=1000 velocity=100
- joint crazyflie_M4_joint: limit lower=-1e+16 upper=1e+16 effort=-1 velocity=-1 -> lower=-1e+16 upper=1e+16 effort=1000 velocity=100

Commit message: CrazySim properly generates the velocity controller topics, used to set the setpoint for each motor

File: crazyflie_description/urdf/crazyflie_basic.urdf (robot description, URDF)
Before this commit: robot crazyflie, 5 links, 4 joints
Links:
- link crazyflie_main_body: geometry collision box size=0.045 0.045 0.03; visual mesh filename=/home/andrea/catkin_ws/src/crazyflie_description/meshes/cra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
- link crazyflie_prop_M1: geometry collision cylinder length=0.005 radius=0.0225; visual mesh filename=/home/andrea/catkin_ws/src/crazyflie_description/meshes/pro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 scale=0.0225 0.0225 0.0225
- link crazyflie_prop_M2: geometry collision cylinder length=0.005 radius=0.0225; visual mesh filename=/home/andrea/catkin_ws/src/crazyflie_description/meshes/pro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 scale=0.0225 0.0225 0.0225
- link crazyflie_prop_M3: geometry collision cylinder length=0.005 radius=0.0225; visual mesh filename=/home/andrea/catkin_ws/src/crazyflie_description/meshes/pro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 scale=0.0225 0.0225 0.0225
- link crazyflie_prop_M4: geometry collision cylinder length=0.005 radius=0.0225; visual mesh filename=/home/andrea/catkin_ws/src/crazyflie_description/meshes/pro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 scale=0.0225 0.0225 0.0225
