Commit message: Added torque due to drag force

File: crazyflie_description/urdf/crazyflie_test_bench.urdf (robot description, URDF)
Before this commit: robot crazyflie, 8 links, 7 joints
Links:
- removed link world
- added link world_link
- link column: mass 1.0 -> 1000.0; geometry collision sphere radius=0.005; visual cylinder length=0.5 radius=0.01
Joints:
- joint fixed_cf_joint: axis (none) -> 1 0 0; limit (none) -> lower=-0.785 upper=0.785 effort=1000 velocity=100; origin xyz=0 0 0.5 rpy=0 0 0 -> xyz=0 0 0.482 rpy=0 0 0; type fixed -> revolute
- joint fixed_column_joint: origin xyz=0 0 0.25 rpy=0 0 0 -> xyz=0 0 0 rpy=0 0 0; parent world -> world_link
